File: ESP8266-07.sch (KiCad schematic (older format))
At the start: 38 parts, among them J1 HEADER_2, J2 HEADER_3, J3 HEADER_3, J4 HEADER_3, J5 HEADER_3, J6 HEADER_3, Q1 BC817-40, Q2 BC817-40, SW1 SW_PUSH, SW2 SW_PUSH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

Commit message: fix
Parts:
- removed U3: AMS1117, symbol AMS1117
- added U3: LM1117-3.3, symbol LM1117-3.3
- C1, C2, C3, C4, C6: footprint (none) -> w_smd_cap:c_1206
- D1, D2, D3: footprint (none) -> LEDs:LED_1206
- U4, U5: symbol Omron_G3MB-202P -> Omron_G3MB-202P-RESCUE-ESP8266-07
Connections:
- wire segments 134 -> 126

Commit message: fix
Parts:
- AC1: renamed from J1; footprint (none) -> w_conn_mkds:mkds_1,5-2
- C5: footprint (none) -> Capacitors_Tantalum_SMD:CP_Tantalum_Case-U_EIA-6032-15_Wave
- F1, F2: footprint (none) -> Fuse_Holders_and_Fuses:Fuse_SMD1206_Reflow
- Flash1: renamed from SW2; footprint (none) -> w_switch:smd_push
- J3, J6: footprint (none) -> w_conn_mkds:mkds_1,5-3
- PIR1: renamed from J2; footprint (none) -> w_pin_strip:pin_strip_2mm_3
- Q1, Q2: footprint TO_SOT_Packages_SMD:SOT-23 -> w_smd_trans:sot23
- R1, R10, R11, R2, R3, R4, R5, R6, R7, R8, R9: footprint (none) -> w_smd_resistors:r_1206
- RV1: footprint (none) -> Varistors:RV_Disc_D7_W3.4_P5
- Res1: renamed from SW1; footprint (none) -> w_switch:smd_push
- SENSOR1: renamed from J5; footprint (none) -> w_pin_strip:pin_strip_2mm_3
- SERIAL1: renamed from J4; footprint (none) -> w_pin_strip:pin_strip_2mm_3
- U1: footprint (none) -> ESP8266:ESP-07v2
- U2: footprint (none) -> makerlab:HLK-PM01
- U3: footprint (none) -> w_smd_trans:sot223; symbol LM1117-3.3 -> LM1117-3.3-RESCUE-ESP8266-07
Connections:
- net +3.3V: now also SENSOR1.2; no longer SENSOR1.1
- net +5V: now also PIR1.2; no longer PIR1.1
- net GND: now also PIR1.1, SENSOR1.1; no longer PIR1.3, SENSOR1.3
- net Lin: now also AC1.1; no longer AC1.2
- net Neu: now also AC1.2; no longer AC1.1
- net PIR: now also PIR1.3; no longer PIR1.2
- net Sensor: now also SENSOR1.3; no longer SENSOR1.2
Other:
- moved on the sheet: AC1
